File: GateMateA1-HDMI-EVB.kicad_sch (KiCad schematic)
At the start: 298 parts, among them Q1 Q12MHz/20pF/10ppm/4P/3.2x2.5mm, U1 CCGM1A1(FBGA-324), U10 RP2040(QFN-56_7x7mm_P0.4mm), U11 TPS62A02ADRLR(SOT-563-6), U12 TPS62A02ADRLR(SOT-563-6), U13 TPS62A02ADRLR(SOT-563-6), U14 TPS62A02ADRLR(SOT-563-6), U15 TPS62A02ADRLR(SOT-563-6), U2 HX7027(SOT-23-3), U3 NA(ZD25WQ16CSIGT(SOIC-8_208mi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, U4 NA(MCP120T-300I/TT(SOT-23-3)), U5 TXB0108PWR(TSSOP-20), U6 TXB0108PWR(TSSOP-20), U7 LY68S3200SLT(SOIC-8_150mil), U8 ZD25WQ16CSIGT(SOIC-8_208mils), U9 LY68S3200SLT(SOIC-8_150mil)

Commit message: Update Schematics
Parts:
- removed VGA1: HDR15-3.08-14.5T/VGA15/14.5mm, OLIMEX_Connectors-FP:VGA15-F(HDR15-3.08-14.5T)_DrillSlot, symbol OLIMEX_Connectors:VGA15-F(CD0515S21J0)
- added ALIN1, ARIN1: TESTPAD, OLIMEX_Other-FP:TEST_PAD_40x70_Round, symbol OLIMEX_OTHER:TESTPAD
- added C127, C132: 22uF/6.3V/20%/X5R/C0603, OLIMEX_RLC-FP:C_0603_5MIL_DWS, symbol OLIMEX_RCL:C
- added C128, C129, C130, C131, C133, C134, C135, C136, C137, C138, C139, C147: 100nF/10V/20%/X5R/C0402, OLIMEX_RLC-FP:C_0402_5MIL_DWS, symbol OLIMEX_RCL:C
- added C140, C141: 33pF/50V/5%/C0G/C0402, OLIMEX_RLC-FP:C_0402_5MIL_DWS, symbol OLIMEX_RCL:C
- added C142, C143, C144: 47nF/50V/10%/X7R/C0402, OLIMEX_RLC-FP:C_0402_5MIL_DWS, symbol OLIMEX_RCL:C
- added C145, C146: 4.7uF/X5R/20%/10V/C0402, OLIMEX_RLC-FP:C_0402_5MIL_DWS, symbol OLIMEX_RCL:C
- added C148: NA(1nF/C0402), OLIMEX_RLC-FP:C_0402_5MIL_DWS, symbol OLIMEX_RCL:C
- added D2: CH213K(SOT23-3), OLIMEX_Diodes-FP:SOT23-3, symbol OLIMEX_Diodes:CH213K(SOT23-3)
- added FUSE1: NA(FSMD035-1206), OLIMEX_Devices-FP:FUSE-1206, symbol OLIMEX_Devices:FSMD035
- added HCEC1, PC0, SCL1, SDA1, SPDIF1, SWC1, SWD2: TESTPAD, OLIMEX_Other-FP:TESTPAD_40-ROUND, symbol OLIMEX_OTHER:TESTPAD
- added HDMI_OUT1: HDMI-SWM-19, OLIMEX_Connectors-FP:HDMI-SWM-19_Paste, symbol OLIMEX_Connectors:HDMI-SWM-19
- added L8, L9: IND/600OHM/2A/UPZ2012E-601-2R0TF/L0805, OLIMEX_RLC-FP:L_0805_5MIL_DWS, symbol OLIMEX_RCL:L
- added Q2: Q24.576MHz/20pF/20ppm/2P/5x3.2mm, OLIMEX_Crystal-FP:HCX-4S_2Pins_5.0x3.2mm_TEST, symbol OLIMEX_Devices:Crystal
- added R80: 1k/1%/R0402, OLIMEX_RLC-FP:R_0402_5MIL_DWS, symbol OLIMEX_RCL:R
- added R81: NA(4.7k/R0402), OLIMEX_RLC-FP:R_0402_5MIL_DWS, symbol OLIMEX_RCL:R
- added R82, R83: 75R/1%/R0402, OLIMEX_RLC-FP:R_0402_5MIL_DWS, symbol OLIMEX_RCL:R
- added R86, R94: NA(10k/R0402), OLIMEX_RLC-FP:R_0402_5MIL_DWS, symbol OLIMEX_RCL:R
- added R87: 0R/R0402/Board_Mounted, OLIMEX_RLC-FP:R_0402_5MIL_0R(Board_Mounted), symbol OLIMEX_RCL:R
- added R88, R89, R90, R91, R92, R93: 10k/R0402, OLIMEX_RLC-FP:R_0402_5MIL_DWS, symbol OLIMEX_RCL:R
- added U16: CV8986(QFN56_7x7mm), OLIMEX_IC-FP:QFN56_7x7_Pitch_0.4mm_EPad_5.4x5.4mm, symbol OLIMEX_IC:CV8986(QFN56)
Connections:
- net +2V5: now also RM1.2, RM1.4, RM1.6, RM3.2, RM3.4, RM3.6, RM3.8; no longer RM1.1.2, RM1.2.2, RM1.3.2, RM3.1.2, RM3.2.2, RM3.3.2, RM3.4.2
- net +5V_USB: now also D2.3 (VI+), FUSE1.1, R92.1, R93.1
- net CFG_MD0: now also RM2.7; no longer RM2.4.1
- net CFG_MD1: now also RM2.5; no longer RM2.3.1
- net CFG_MD2: now also RM2.3; no longer RM2.2.1
- net CFG_MD3: now also RM2.1; no longer RM2.1.1
- net FPGA_SPI_D0: now also RM3.1; no longer RM3.1.1
- net FPGA_SPI_D1: now also RM3.5; no longer RM3.3.1
- net FPGA_SPI_D2: now also RM3.3; no longer RM3.2.1
- net FPGA_SPI_D3: now also RM3.7; no longer RM3.4.1
- net GND: now also RM1.8, RM2.2, RM2.4, RM2.6, RM2.8, C127.2, C128.2, C129.2, C130.2, C131.2, C132.2, C133.2, C134.2, C135.2, C136.2, C137.2, C138.2, C139.2, C140.2, C141.2, C147.1, D2.1 (GND), HDMI_OUT1.11, HDMI_OUT1.17, HDMI_OUT1.2, HDMI_OUT1.20, HDMI_OUT1.21, HDMI_OUT1.22, HDMI_OUT1.23, HDMI_OUT1.5, HDMI_OUT1.8, R80.1, R87.2, R88.2, R91.2, R94.1, U16.1 (AVSS), U16.14 (VSS), U16.16 (AVSS), U16.22 (AVSS), U16.28 (AVSS), U16.32 (DVSS), U16.36 (PA11), U16.37 (PA12), U16.45 (GND), U16.49 (AVSS), U16.53 (AVSS), U16.56 (AVSS), U16.57 (EPAD); no longer RM1.4.2, RM2.1.2, RM2.2.2, RM2.3.2, RM2.4.2
- net GPIO16\JTAG_TDI: now also RM1.5; no longer RM1.3.1
- net GPIO17\JTAG_TDO: now also RM1.3; no longer RM1.2.1
- net GPIO18\JTAG_TCK: now also RM1.7; no longer RM1.4.1
- net GPIO19\JTAG_TMS: now also RM1.1; no longer RM1.1.1
- net VGA_HSync: now also R83.2
- net VGA_VSync: now also R82.2
- net BLUE_IN: now reaches R41.1, R42.1, R43.1, R44.1, TVS1.2 (IO2)
- net BLUE_IN: now also C144.1
- net GREEN_IN: now reaches R37.1, R38.1, R39.1, R40.1, TVS2.2 (IO2)
- net GREEN_IN: now also C143.1, C148.1
- net RED_IN: now reaches R32.1, R33.1, R34.1, R35.1, TVS3.2 (IO2)
- net RED_IN: now also C142.1
- new net: HCEC1.1 (Pad), HDMI_OUT1.13
- new net: R82.1, U16.41 (VS_IN)
- new net: SWC1.1 (Pad), U16.39 (SWCLK)
- new net: C140.1, Q2.1, U16.30 (XTI)
- new net: C146.1, R90.1, R91.1
- new net: PC0.1 (Pad), R87.1, U16.10 (PC0)
- new net: R83.1, U16.40 (HS_IN)
- new net: ALIN1.1 (Pad), R90.2
- new net: C145.1, R88.1, R89.1
- new net: C145.2, U16.2 (ARIN)
- new net: C141.1, Q2.2, U16.31 (XTO)
- new net: C142.2, U16.55 (RIN)
- new net: C144.2, U16.48 (BIN)
- new net: SPDIF1.1 (Pad), U16.5 (SPDIF)
- new net: SWD2.1 (Pad), U16.38 (SWDIO)
- new net: R80.2, U16.15 (REXT)
- new net: C147.2, R86.1, U16.11 (NRST)
- new net: C143.2, U16.51 (GIN)
- new net: ARIN1.1 (Pad), R89.2
- new net: SDA1.1 (Pad), U16.34 (SDA)
- new net: C148.2, R81.2
- new net: C146.2, U16.3 (ALIN)
- new net: SCL1.1 (Pad), U16.33 (SCL)
- new net: R81.1, U16.50 (SOG0)
- new net +1.8V: C130.1, C131.1, C138.1, C139.1, L9.1, U16.19 (AV18H), U16.25 (AV18H), U16.35 (DVDD18), U16.6 (DVDD18)
- new net +3.3V: C134.1, C135.1, C136.1, C137.1, L8.1, R86.2, U16.12 (VDD33), U16.13 (VDD33), U16.29 (DV33), U16.42 (DV33)
- new net AV18: C132.1, C133.1, L9.2, U16.52 (AV18)
- new net AV33: C127.1, C128.1, C129.1, L8.2, U16.4 (AV33), U16.54 (AV33)
- new net HDMI_5V: D2.2 (VO-), FUSE1.2, HDMI_OUT1.18
- new net HDMI_HPD: HDMI_OUT1.19, R94.2, U16.7 (HPD)
- new net HDMI_SCL: HDMI_OUT1.15, R92.2, U16.9 (DDC_SCL)
- new net HDMI_SDA: HDMI_OUT1.16, R93.2, U16.8 (DDC_SDA)
- new net HDMI_TX0+: HDMI_OUT1.7, U16.21 (TX0P)
- new net HDMI_TX0-: HDMI_OUT1.9, U16.20 (TX0N)
- new net HDMI_TX1+: HDMI_OUT1.4, U16.24 (TX1P)
- new net HDMI_TX1-: HDMI_OUT1.6, U16.23 (TX1N)
- new net HDMI_TX2+: HDMI_OUT1.1, U16.27 (TX2P)
- new net HDMI_TX2-: HDMI_OUT1.3, U16.26 (TX2N)
- new net HDMI_TXC+: HDMI_OUT1.10, U16.18 (TXCP)
- new net HDMI_TXC-: HDMI_OUT1.12, U16.17 (TXCN)
Other:
- note added: "VGA2HDMI - CV8986"
- company: OLIMEX LTD. -> Amr Badr
- title: GateMateA1-EVB -> GateMateA1-HDMI-EVB

Commit message: Fixed HDMI Bus warnings
Parts:
- UEXT1: Note (none) -> PB-Free
Connections:
- net +1.8V is gone; now on net +1V8: C130.1, C131.1, C138.1, C139.1, L9.1, U16.19 (AV18H), U16.25 (AV18H), U16.35 (DVDD18), U16.6 (DVDD18)
- net +3.3V is gone; now on net +3V3: C134.1, C135.1, C136.1, C137.1, L8.1, R86.2, U16.12 (VDD33), U16.13 (VDD33), U16.29 (DV33), U16.42 (DV33)
Changed lines of the file:
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@@
 		)
 	)
+	(bus_alias "HDMI-BUS"
+		(members "HDMI_TX2+" "HDMI_TX2-" "HDMI_TX1+" "HDMI_TX1-" "HDMI_TX0+" "HDMI_TX0-"
+			"HDMI_SCL" "HDMI_SDA" "HDMI_HPD" "HDMI_TXC+" "HDMI_TXC-"
+		)
+	)
 	(bus_alias "Main-BUS"
 		(members "GPIO[0..11]" "GPIO12\\DBG-UART_TX" "GPIO13\\DBG-UART_RX" "GPIO[14..15]"
@@
 		)
 	)
+	(label "{HDMI-BUS}"
+		(at 421.64 410.21 90)
+		(effects
+			(font
+				(size 2.54 2.54)
+				(thickness 0.508)
+				(bold yes)
+				(color 194 0 0 1)
+			)
+			(justify left bottom)
+		)
+	)
 	(label "NB_B3"
 		(at 266.7 289.56 0)
@@
 			)
 		)
-		(property "Value" "+1.8V"
+		(property "Value" "+1V8"
 			(at 576.58 317.5 90)
 			(effects
@@
 			)
 		)
-		(property "Value" "+1.8V"
+		(property "Value" "+1V8"
 			(at 576.58 309.88 90)
 			(effects
@@
 			)
 		)
-		(property "Value" "+1.8V"
+		(property "Value" "+1V8"
 			(at 576.58 358.14 90)
 			(effects
@@
 			)
 		)
-		(property "Value" "+3.3V"
+		(property "Value" "+3V3"
 			(at 579.755 345.44 90)
 			(effects
@@
 			)
 		)
-		(property "Value" "+3.3V"
+		(property "Value" "+3V3"
 			(at 433.705 370.84 90)
 			(effects
@@
 			)
 		)
-		(property "Value" "+3.3V"
+		(property "Value" "+3V3"
 			(at 579.755 299.72 90)
 			(effects
@@
 			)
 		)
-		(property "Description" ""
+		(property "Description" "Connector 10 pins 2x5"
 			(at 45.72 266.7 0)
 			(effects
@@
 					(size 1.27 1.27)
 				)
+				(hide yes)
 			)
 		)
@@
 				)
 				(hide yes)
+			)
+		)
+		(property "Note" "PB-Free"
+			(at 45.72 284.48 0)
+			(effects
+				(font
+					(size 1.27 1.27)
+				)
+				(hide yes)

Commit message: Revert RA1206_(4X0603)_4B8_xx Pins
Connections:
- net +2V5: now also RM1.1.2, RM1.2.2, RM1.3.2, RM3.1.2, RM3.2.2, RM3.3.2, RM3.4.2; no longer RM1.2, RM1.4, RM1.6, RM3.2, RM3.4, RM3.6, RM3.8
- net CFG_MD0: now also RM2.4.1; no longer RM2.7
- net CFG_MD1: now also RM2.3.1; no longer RM2.5
- net CFG_MD2: now also RM2.2.1; no longer RM2.3
- net CFG_MD3: now also RM2.1.1; no longer RM2.1
- net FPGA_SPI_D0: now also RM3.1.1; no longer RM3.1
- net FPGA_SPI_D1: now also RM3.3.1; no longer RM3.5
- net FPGA_SPI_D2: now also RM3.2.1; no longer RM3.3
- net FPGA_SPI_D3: now also RM3.4.1; no longer RM3.7
- net GND: now also RM1.4.2, RM2.1.2, RM2.2.2, RM2.3.2, RM2.4.2; no longer RM1.8, RM2.2, RM2.4, RM2.6, RM2.8
- net GPIO16\JTAG_TDI: now also RM1.3.1; no longer RM1.5
- net GPIO17\JTAG_TDO: now also RM1.2.1; no longer RM1.3
- net GPIO18\JTAG_TCK: now also RM1.4.1; no longer RM1.7
- net GPIO19\JTAG_TMS: now also RM1.1.1; no longer RM1.1
Changed lines of the file:
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@@
 	)
 	(symbol
-		(lib_name "RA1206_(4x0603)_4B8_Smashed_6")
 		(lib_id "OLIMEX_RCL:RA1206_(4x0603)_4B8_Smashed")
 		(at 142.24 176.53 0)
@@
 			)
 		)
-		(pin "4"
+		(pin "2.2"
 		)
-		(pin "1"
+		(pin "1.2"
 		)
-		(pin "5"
+		(pin "4.1"
 		)
-		(pin "6"
+		(pin "3.2"
 		)
-		(pin "2"
+		(pin "4.2"
 		)
-		(pin "7"
+		(pin "3.1"
 		)
-		(pin "8"
+		(pin "1.1"
 		)
-		(pin "3"
+		(pin "2.1"
 		)
 		(instances
@@
 	)
 	(symbol
-		(lib_name "RA1206_(4x0603)_4B8_Smashed_5")
 		(lib_id "OLIMEX_RCL:RA1206_(4x0603)_4B8_Smashed")
 		(at 142.24 171.45 0)
@@
 			)
 		)
-		(pin "6"
+		(pin "4.1"
 		)
-		(pin "5"
+		(pin "3.2"
 		)
-		(pin "8"
+		(pin "4.2"
 		)
-		(pin "7"
+		(pin "1.1"
 		)
-		(pin "2"
+		(pin "2.2"
 		)
-		(pin "4"
+		(pin "3.1"
 		)
-		(pin "1"
+		(pin "1.2"
 		)
-		(pin "3"
+		(pin "2.1"
 		)
 		(instances
@@
 			)
 		)
-		(pin "8"
+		(pin "3.1"
 		)
-		(pin "7"
+		(pin "2.1"
 		)
-		(pin "6"
+		(pin "1.1"
 		)
-		(pin "2"
+		(pin "2.2"
 		)
-		(pin "5"
+		(pin "1.2"
 		)
-		(pin "1"
+		(pin "4.1"
 		)
-		(pin "3"
+		(pin "4.2"
 		)
-		(pin "4"
+		(pin "3.2"
 		)
 		(instances
@@
 	)
 	(symbol
-		(lib_name "RA1206_(4x0603)_4B8_Smashed_7")
 		(lib_id "OLIMEX_RCL:RA1206_(4x0603)_4B8_Smashed")
 		(at 142.24 173.99 0)
@@
 			)
 		)
-		(pin "8"
+		(pin "4.1"
 		)
-		(pin "2"
+		(pin "2.1"
 		)
-		(pin "4"
+		(pin "1.2"
 		)
-		(pin "7"
+		(pin "3.1"
 		)
-		(pin "1"
+		(pin "1.1"
 		)
-		(pin "6"
+		(pin "2.2"
 		)
-		(pin "5"
+		(pin "4.2"
 		)
-		(pin "3"
+		(pin "3.2"
 		)
 		(instances
@@
 			)
 		)
-		(pin "4"
+		(pin "4.1"
 		)
-		(pin "5"
+		(pin "3.1"
 		)
-		(pin "1"
+		(pin "4.2"
 		)
-		(pin "7"
+		(pin "3.2"
 		)
-		(pin "8"
+		(pin "1.1"
 		)
-		(pin "6"
+		(pin "2.2"
 		)
-		(pin "3"
+		(pin "1.2"
 		)
-		(pin "2"
+		(pin "2.1"
 		)
 		(instances
@@
 			)
 		)
-		(pin "1"
+		(pin "4.2"
 		)
-		(pin "5"
+		(pin "3.2"
 		)
-		(pin "4"
+		(pin "2.2"
 		)
-		(pin "8"
+		(pin "3.1"
 		)
-		(pin "6"
+		(pin "1.2"
 		)
-		(pin "3"
+		(pin "1.1"
 		)
-		(pin "2"
+		(pin "2.1"
 		)
-		(pin "7"
+		(pin "4.1"
 		)
 		(instances
@@
 			)
 		)
-		(pin "5"
+		(pin "1.2"
 		)
-		(pin "2"
+		(pin "2.1"
 		)
-		(pin "7"
+		(pin "3.1"
 		)
-		(pin "1"
+		(pin "4.2"
 		)
-		(pin "6"
+		(pin "4.1"
 		)
-		(pin "4"
+		(pin "3.2"
 		)
-		(pin "8"
+		(pin "1.1"
 		)
-		(pin "3"
+		(pin "2.2"
 		)
 		(instances
@@
 			)
 		)
-		(pin "3"
+		(pin "4.1"
 		)
-		(pin "4"
+		(pin "2.1"
 		)
-		(pin "6"
+		(pin "1.2"
 		)
-		(pin "5"
+		(pin "1.1"
 		)
-		(pin "2"
+		(pin "3.1"
 		)
-		(pin "7"
+		(pin "4.2"
 		)
-		(pin "1"
+		(pin "3.2"
 		)
-		(pin "8"
+		(pin "2.2"
 		)
 		(instances
@@
 	)
 	(symbol
-		(lib_name "RA1206_(4x0603)_4B8_Smashed_8")
 		(lib_id "OLIMEX_RCL:RA1206_(4x0603)_4B8_Smashed")
 		(at 142.24 168.91 0)
@@
 			)
 		)
-		(pin "5"
+		(pin "2.1"
 		)
-		(pin "6"
+		(pin "1.2"
 		)
-		(pin "7"
+		(pin "1.1"
 		)
-		(pin "1"
+		(pin "4.1"
 		)
-		(pin "2"
+		(pin "3.2"
 		)
-		(pin "3"
+		(pin "3.1"
 		)
-		(pin "4"
+		(pin "4.2"
 		)
-		(pin "8"
+		(pin "2.2"
 		)
 		(instances
@@
 			)
 		)
-		(pin "7"
+		(pin "1.2"
 		)
-		(pin "5"
+		(pin "2.1"
 		)
-		(pin "3"
+		(pin "4.2"
 		)
-		(pin "8"
+		(pin "1.1"
 		)
-		(pin "1"
+		(pin "3.1"
 		)
-		(pin "6"
+		(pin "2.2"
 		)
-		(pin "2"
+		(pin "3.2"
 		)
-		(pin "4"
+		(pin "4.1"
 		)
 		(instances
@@
 			)
 		)
-		(pin "2"
+		(pin "3.2"
 		)
-		(pin "5"
+		(pin "1.2"
 		)
-		(pin "1"
+		(pin "4.1"
 		)
-		(pin "8"
+		(pin "3.1"
 		)
-		(pin "6"
+		(pin "4.2"
 		)
-		(pin "4"
+		(pin "2.2"
 		)
-		(pin "7"
+		(pin "1.1"
 		)
-		(pin "3"
+		(pin "2.1"
 		)
 		(instances
@@
 			)
 		)
-		(pin "4"
+		(pin "3.2"
 		)
-		(pin "2"
+		(pin "1.1"
 		)
-		(pin "3"
+		(pin "2.1"
 		)
-		(pin "5"
+		(pin "2.2"
 		)
-		(pin "1"
+		(pin "4.1"
 		)
-		(pin "6"
+		(pin "1.2"
 		)
-		(pin "8"
+		(pin "3.1"
 		)
-		(pin "7"
+		(pin "4.2"
 		)
 		(instances
